File: Peripherals.sch (KiCad schematic (older format))
At the start: 26 parts, among them J10 TEST_1P, J11 TEST_1P, J12 Micro_SD_Card, J13 TEST_1P, J14 TEST_1P, J15 TEST_1P, J16 TEST_1P, J17 TEST_1P, J4 TEST_1P, J5 TEST_1P, J6 TEST_1P, J7 TEST_1P, J8 TEST_1P, J9 TEST_1P, U6 MS5607, U7 LSM9DS1

Commit message: Bring schematic in line with PCB. Previous update broke this.
Parts:
- C27, C28, C29, C30, C31, C32: footprint Capacitor_SMD:C_0603_1608Metric -> Capacitors_SMD:C_0603
- J10, J11, J13, J14, J15, J16, J17, J4, J5, J6, J7, J8, J9: footprint TestPoint:TestPoint_Pad_D2.0mm -> Connectors_TestPoints:Test_Point_Pad_d1.5mm
- R10, R11, R12, R9: footprint Resistor_SMD:R_0603_1608Metric -> Resistors_SMD:R_0603

Commit message: Changes based on review reccommemdations
Parts:
- added C36: 10u, Capacitors_SMD:C_0603, symbol C
Connections:
- net +3V3: now also C36.1
- net GND: now also C36.2
Changed lines of the file:
@@
 Text GLabel 2075 4800 0    39   Input ~ 0
 SPI3_SCK
-Text GLabel 1175 4500 0    39   Input ~ 0
+Text GLabel 1490 4500 0    39   Input ~ 0
 SD1_~CS
 Text GLabel 1770 4600 0    39   Input ~ 0
 SPI3_MOSI
 $Comp
-L GND #PWR037
+L GND #PWR036
 U 1 1 5A079410
 P 2350 5200
-F 0 "#PWR037" H 2350 4950 50  0001 C CNN
+F 0 "#PWR036" H 2350 4950 50  0001 C CNN
 F 1 "GND" H 2350 5050 50  0000 C CNN
 F 2 "" H 2350 5200 50  0001 C CNN
@@
 $EndComp
 $Comp
-L +3.3V #PWR038
+L +3.3V #PWR037
 U 1 1 5A1097BB
 P 1865 1575
-F 0 "#PWR038" H 1865 1425 50  0001 C CNN
+F 0 "#PWR037" H 1865 1425 50  0001 C CNN
 F 1 "+3.3V" H 1865 1715 50  0000 C CNN
 F 2 "" H 1865 1575 50  0001 C CNN
@@
 $EndComp
 $Comp
-L GND #PWR039
+L GND #PWR038
 U 1 1 5A109D13
 P 1865 2125
-F 0 "#PWR039" H 1865 1875 50  0001 C CNN
+F 0 "#PWR038" H 1865 1875 50  0001 C CNN
 F 1 "GND" H 1865 1975 50  0000 C CNN
 F 2 "" H 1865 2125 50  0001 C CNN
@@
 $EndComp
 $Comp
-L GND #PWR040
+L GND #PWR039
 U 1 1 5A1CEA47
 P 7570 1550
-F 0 "#PWR040" H 7570 1300 50  0001 C CNN
+F 0 "#PWR039" H 7570 1300 50  0001 C CNN
 F 1 "GND" H 7570 1400 50  0000 C CNN
 F 2 "" H 7570 1550 50  0001 C CNN
@@
 $EndComp
 $Comp
-L GND #PWR041
+L GND #PWR040
 U 1 1 5A1CED55
 P 8595 1550
-F 0 "#PWR041" H 8595 1300 50  0001 C CNN
+F 0 "#PWR040" H 8595 1300 50  0001 C CNN
 F 1 "GND" H 8595 1400 50  0000 C CNN
 F 2 "" H 8595 1550 50  0001 C CNN
@@
 $EndComp
 $Comp
-L GND #PWR042
+L GND #PWR041
 U 1 1 5A1CF4A7
 P 6445 3125
-F 0 "#PWR042" H 6445 2875 50  0001 C CNN
+F 0 "#PWR041" H 6445 2875 50  0001 C CNN
 F 1 "GND" H 6445 2975 50  0000 C CNN
 F 2 "" H 6445 3125 50  0001 C CNN
@@
 $EndComp
 $Comp
-L GND #PWR043
+L GND #PWR042
 U 1 1 5A1CF5D2
 P 6445 3400
-F 0 "#PWR043" H 6445 3150 50  0001 C CNN
+F 0 "#PWR042" H 6445 3150 50  0001 C CNN
 F 1 "GND" H 6445 3250 50  0000 C CNN
 F 2 "" H 6445 3400 50  0001 C CNN
@@
 $EndComp
 $Comp
-L GND #PWR044
+L GND #PWR043
 U 1 1 5A1CF685
 P 7895 3475
-F 0 "#PWR044" H 7895 3225 50  0001 C CNN
+F 0 "#PWR043" H 7895 3225 50  0001 C CNN
 F 1 "GND" H 7895 3325 50  0000 C CNN
 F 2 "" H 7895 3475 50  0001 C CNN
@@
 $EndComp
 $Comp
-L +3.3V #PWR045
+L +3.3V #PWR044
 U 1 1 5A1D43CB
 P 9120 1625
-F 0 "#PWR045" H 9120 1475 50  0001 C CNN
+F 0 "#PWR044" H 9120 1475 50  0001 C CNN
 F 1 "+3.3V" H 9120 1765 50  0000 C CNN
 F 2 "" H 9120 1625 50  0001 C CNN
@@
 $EndComp
 $Comp
-L +3.3V #PWR046
+L +3.3V #PWR045
 U 1 1 5A223437
 P 8070 1175
-F 0 "#PWR046" H 8070 1025 50  0001 C CNN
+F 0 "#PWR045" H 8070 1025 50  0001 C CNN
 F 1 "+3.3V" H 8070 1315 50  0000 C CNN
 F 2 "" H 8070 1175 50  0001 C CNN
@@
 $EndComp
 $Comp
-L +3.3V #PWR047
+L +3.3V #PWR046
 U 1 1 5A24A5D9
 P 2200 4125
-F 0 "#PWR047" H 2200 3975 50  0001 C CNN
+F 0 "#PWR046" H 2200 3975 50  0001 C CNN
 F 1 "+3.3V" H 2200 4265 50  0000 C CNN
 F 2 "" H 2200 4125 50  0001 C CNN
@@
 $EndComp
 $Comp
-L GND #PWR048
+L GND #PWR047
 U 1 1 5A36B036
 P 5315 5310
-F 0 "#PWR048" H 5315 5060 50  0001 C CNN
+F 0 "#PWR047" H 5315 5060 50  0001 C CNN
 F 1 "GND" H 5315 5160 50  0000 C CNN
 F 2 "" H 5315 5310 50  0001 C CNN
@@
 A/G_~CS
 $Comp
-L +3.3V #PWR049
+L +3.3V #PWR048
 U 1 1 5A1D497E
 P 6295 1725
-F 0 "#PWR049" H 6295 1575 50  0001 C CNN
+F 0 "#PWR048" H 6295 1575 50  0001 C CNN
 F 1 "+3.3V" H 6295 1865 50  0000 C CNN
 F 2 "" H 6295 1725 50  0001 C CNN
@@
 	2350 4900 2350 5200
 Wire Wire Line
-	1625 4125 2200 4125
+	1055 4125 2200 4125
 Wire Wire Line
 	1865 1750 2115 1750
@@
 	6195 2225 7195 2225
 Wire Wire Line
-	7195 2325 6195 2325
+	6195 2325 7195 2325
 Wire Wire Line
 	7195 2625 6170 2625
@@
 	1865 1575 1865 1750
 Wire Wire Line
-	1175 4500 3465 4500
+	1490 4500 3465 4500
 Wire Wire Line
 	1625 4425 1625 4500
@@
 	6605 2170 6605 2525
 Connection ~ 6605 2525
+$Comp
+L C C36
+U 1 1 5AF5B0B5
+P 1055 4280
+F 0 "C36" H 1080 4380 50  0000 L CNN
+F 1 "10u" H 1080 4180 50  0000 L CNN
+F 2 "Capacitors_SMD:C_0603" H 1093 4130 50  0001 C CNN
+F 3 "" H 1055 4280 50  0001 C CNN
+	1    1055 4280
+	1    0    0    -1
+$EndComp
+Wire Wire Line
+	1055 4125 1055 4130
+Connection ~ 1625 4125
+$Comp
+L GND #PWR049
+U 1 1 5AF5B75D
+P 1055 4490
+F 0 "#PWR049" H 1055 4240 50  0001 C CNN
+F 1 "GND" H 1055 4340 50  0000 C CNN
+F 2 "" H 1055 4490 50  0001 C CNN
+F 3 "" H 1055 4490 50  0001 C CNN
+	1    1055 4490
+	1    0    0    -1
+$EndComp
+Wire Wire Line
+	1055 4430 1055 4490
 $EndSCHEMATC

Commit message: Final design published. Gerbers and PDF schematic generated
Parts:
- J12: footprint SOAR_Library:Conn,Molex,Hinged_microSD -> SOAR_Kicad_Library:Conn,Molex,Hinged_microSD
Changed lines of the file:
@@
 F 0 "J12" H 3715 5300 50  0000 C CNN
 F 1 "Micro_SD_Card" H 5015 5300 50  0000 R CNN
-F 2 "SOAR_Library:Conn,Molex,Hinged_microSD" H 5515 5000 50  0001 C CNN
+F 2 "SOAR_Kicad_Library:Conn,Molex,Hinged_microSD" H 5515 5000 50  0001 C CNN
 F 3 "http://www.molex.com/pdm_docs/sd/472192001_sd.pdf" H 4365 4700 50  0001 C CNN
 F 4 "0472192001" H 4365 4700 60  0001 C CNN "Digikey"
@@
 SPI3_MOSI
 $Comp
-L GND #PWR036
+L GND #PWR038
 U 1 1 5A079410
 P 2350 5200
-F 0 "#PWR036" H 2350 4950 50  0001 C CNN
+F 0 "#PWR038" H 2350 4950 50  0001 C CNN
 F 1 "GND" H 2350 5050 50  0000 C CNN
 F 2 "" H 2350 5200 50  0001 C CNN
@@
 $EndComp
 $Comp
-L +3.3V #PWR037
+L +3.3V #PWR039
 U 1 1 5A1097BB
 P 1865 1575
-F 0 "#PWR037" H 1865 1425 50  0001 C CNN
+F 0 "#PWR039" H 1865 1425 50  0001 C CNN
 F 1 "+3.3V" H 1865 1715 50  0000 C CNN
 F 2 "" H 1865 1575 50  0001 C CNN
@@
 $EndComp
 $Comp
-L GND #PWR038
+L GND #PWR040
 U 1 1 5A109D13
 P 1865 2125
-F 0 "#PWR038" H 1865 1875 50  0001 C CNN
+F 0 "#PWR040" H 1865 1875 50  0001 C CNN
 F 1 "GND" H 1865 1975 50  0000 C CNN
 F 2 "" H 1865 2125 50  0001 C CNN
@@
 $EndComp
 $Comp
-L GND #PWR039
+L GND #PWR041
 U 1 1 5A1CEA47
 P 7570 1550
-F 0 "#PWR039" H 7570 1300 50  0001 C CNN
+F 0 "#PWR041" H 7570 1300 50  0001 C CNN
 F 1 "GND" H 7570 1400 50  0000 C CNN
 F 2 "" H 7570 1550 50  0001 C CNN
@@
 $EndComp
 $Comp
-L GND #PWR040
+L GND #PWR042
 U 1 1 5A1CED55
 P 8595 1550
-F 0 "#PWR040" H 8595 1300 50  0001 C CNN
+F 0 "#PWR042" H 8595 1300 50  0001 C CNN
 F 1 "GND" H 8595 1400 50  0000 C CNN
 F 2 "" H 8595 1550 50  0001 C CNN
@@
 $EndComp
 $Comp
-L GND #PWR041
+L GND #PWR043
 U 1 1 5A1CF4A7
 P 6445 3125
-F 0 "#PWR041" H 6445 2875 50  0001 C CNN
+F 0 "#PWR043" H 6445 2875 50  0001 C CNN
 F 1 "GND" H 6445 2975 50  0000 C CNN
 F 2 "" H 6445 3125 50  0001 C CNN
@@
 $EndComp
 $Comp
-L GND #PWR042
+L GND #PWR044
 U 1 1 5A1CF5D2
 P 6445 3400
-F 0 "#PWR042" H 6445 3150 50  0001 C CNN
+F 0 "#PWR044" H 6445 3150 50  0001 C CNN
 F 1 "GND" H 6445 3250 50  0000 C CNN
 F 2 "" H 6445 3400 50  0001 C CNN
@@
 $EndComp
 $Comp
-L GND #PWR043
+L GND #PWR045
 U 1 1 5A1CF685
 P 7895 3475
-F 0 "#PWR043" H 7895 3225 50  0001 C CNN
+F 0 "#PWR045" H 7895 3225 50  0001 C CNN
 F 1 "GND" H 7895 3325 50  0000 C CNN
 F 2 "" H 7895 3475 50  0001 C CNN
@@
 $EndComp
 $Comp
-L +3.3V #PWR044
+L +3.3V #PWR046
 U 1 1 5A1D43CB
 P 9120 1625
-F 0 "#PWR044" H 9120 1475 50  0001 C CNN
+F 0 "#PWR046" H 9120 1475 50  0001 C CNN
 F 1 "+3.3V" H 9120 1765 50  0000 C CNN
 F 2 "" H 9120 1625 50  0001 C CNN
@@
 $EndComp
 $Comp
-L +3.3V #PWR045
+L +3.3V #PWR047
 U 1 1 5A223437
 P 8070 1175
-F 0 "#PWR045" H 8070 1025 50  0001 C CNN
+F 0 "#PWR047" H 8070 1025 50  0001 C CNN
 F 1 "+3.3V" H 8070 1315 50  0000 C CNN
 F 2 "" H 8070 1175 50  0001 C CNN
@@
 $EndComp
 $Comp
-L +3.3V #PWR046
+L +3.3V #PWR048
 U 1 1 5A24A5D9
 P 2200 4125
-F 0 "#PWR046" H 2200 3975 50  0001 C CNN
+F 0 "#PWR048" H 2200 3975 50  0001 C CNN
 F 1 "+3.3V" H 2200 4265 50  0000 C CNN
 F 2 "" H 2200 4125 50  0001 C CNN
@@
 $EndComp
 $Comp
-L GND #PWR047
+L GND #PWR049
 U 1 1 5A36B036
 P 5315 5310
-F 0 "#PWR047" H 5315 5060 50  0001 C CNN
+F 0 "#PWR049" H 5315 5060 50  0001 C CNN
 F 1 "GND" H 5315 5160 50  0000 C CNN
 F 2 "" H 5315 5310 50  0001 C CNN
@@
 A/G_~CS
 $Comp
-L +3.3V #PWR048
+L +3.3V #PWR050
 U 1 1 5A1D497E
 P 6295 1725
-F 0 "#PWR048" H 6295 1575 50  0001 C CNN
+F 0 "#PWR050" H 6295 1575 50  0001 C CNN
 F 1 "+3.3V" H 6295 1865 50  0000 C CNN
 F 2 "" H 6295 1725 50  0001 C CNN
@@
 Connection ~ 1625 4125
 $Comp
-L GND #PWR049
+L GND #PWR051
 U 1 1 5AF5B75D
 P 1055 4490
-F 0 "#PWR049" H 1055 4240 50  0001 C CNN
+F 0 "#PWR051" H 1055 4240 50  0001 C CNN
 F 1 "GND" H 1055 4340 50  0000 C CNN
 F 2 "" H 1055 4490 50  0001 C CNN
